File: layouts/adapter/adapter.kicad_pcb (KiCad board)
At the start: 2 copper layers, 10 parts

Commit message: wip
Connections:
- J1 pad B6: B6 -> D_plus
- J1 pad B7: B7 -> D_minus
Changed lines of the file:
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@@
     (net 4 "A8")
     (net 5 "esd-net-5")
-    (net 6 "D_minus")
     (net 7 "VDH")
     (net 8 "POGO_SWDIO")
-    (net 9 "D_plus")
     (net 10 "AI4")
     (net 11 "esd-net-4")
@@
     (net 31 "esd-net-1")
     (net 32 "AI2")
-    (net 33 "B7")
     (net 34 "P1_period_11")
     (net 35 "ADAPTER_SWDIO")
@@
     (net 40 "P1_period_09")
     (net 41 "esd-net-0")
-    (net 42 "B6")
     (net 43 "POGO_UART_RX")
     (net 44 "AI6")
@@
     (net 57 "footprint-net-1")
     (net 58 "POGO_I2C_SCL")
+    (net 59 "D_plus")
+    (net 60 "D_minus")
     (footprint "Samsung_Electro_Mechanics_CL05A105KA5NQNC:C0402"
         (layer "F.Cu")
@@
             (size 0.9 2)
             (layers "F.Cu" "F.Paste" "F.Mask")
-            (net 9 "D_plus")
+            (net 59 "D_plus")
         )
         (pad "30" smd rect
@@
             (size 0.9 2)
             (layers "F.Cu" "F.Paste" "F.Mask")
-            (net 6 "D_minus")
+            (net 60 "D_minus")
         )
         (pad "28" smd rect
@@
             (size 0.3 1.3)
             (layers "F.Cu" "F.Paste" "F.Mask")
-            (net 33 "B7")
+            (net 60 "D_minus")
         )
         (pad "A6" smd rect
@@
             (size 0.3 1.3)
             (layers "F.Cu" "F.Paste" "F.Mask")
-            (net 9 "D_plus")
+            (net 59 "D_plus")
         )
         (pad "A7" smd rect
@@
             (size 0.3 1.3)
             (layers "F.Cu" "F.Paste" "F.Mask")
-            (net 6 "D_minus")
+            (net 60 "D_minus")
         )
         (pad "B6" smd rect
@@
             (size 0.3 1.3)
             (layers "F.Cu" "F.Paste" "F.Mask")
-            (net 42 "B6")
+            (net 59 "D_plus")
         )
         (pad "A8" smd rect
