File: layouts/adapter/adapter.kicad_pcb (KiCad board)
At the start: 2 copper layers, 10 parts

Commit message: wip
Parts:
- added C10: 100nF ±10% X5R, Murata_Electronics_GRM033R60J104KE19D:C0201, F.Cu at (0.00, -70.0)
- added C11: 100nF ±10% X5R, Murata_Electronics_GRM033R60J104KE19D:C0201, F.Cu at (0.00, -80.0)
- added C12: 100nF ±10% X5R, Murata_Electronics_GRM033R60J104KE19D:C0201, F.Cu at (0.00, -90.0)
- added C13: 2.2µF ±20% 6.3V X5R, Samsung_Electro_Mechanics_CL05A225MQ5NSNC:C0402, F.Cu at (0.00, -100.0)
- added C14: 100nF ±10% X5R, Murata_Electronics_GRM033R60J104KE19D:C0201, F.Cu at (0.00, -110.0)
- added C15: 100nF ±10% X5R, Murata_Electronics_GRM033R60J104KE19D:C0201, F.Cu at (0.00, -120.0)
- added C16: 100nF ±10% X5R, Murata_Electronics_GRM033R60J104KE19D:C0201, F.Cu at (0.00, -130.0)
- added C17: 100nF ±10% X5R, Murata_Electronics_GRM033R60J104KE19D:C0201, F.Cu at (0.00, -140.0)
- added C18: 10µF ±10% 10V X5R, Samsung_Electro_Mechanics_CL10A106KP8NNNC:C0603, F.Cu at (0.00, -150.0)
- added C19: 10µF ±10% 10V X5R, Samsung_Electro_Mechanics_CL10A106KP8NNNC:C0603, F.Cu at (0.00, -160.0)
- added C20: 1µF ±10% 25V X5R, Samsung_Electro_Mechanics_CL05A105KA5NQNC:C0402, F.Cu at (0.00, -170.0)
- added C21: 10µF ±10% 10V X5R, Samsung_Electro_Mechanics_CL10A106KP8NNNC:C0603, F.Cu at (0.00, -180.0)
- added C5: , DNP_CAP_0201:DNP_CAP_0201, F.Cu at (0.00, -20.0)
- added C6: , DNP_CAP_0201:DNP_CAP_0201, F.Cu at (0.00, -30.0)
- added C7: 100nF ±10% X5R, Murata_Electronics_GRM033R60J104KE19D:C0201, F.Cu at (0.00, -40.0)
- added C8: 100nF ±10% X5R, Murata_Electronics_GRM033R60J104KE19D:C0201, F.Cu at (0.00, -50.0)
- added C9: 100nF ±10% X5R, Murata_Electronics_GRM033R60J104KE19D:C0201, F.Cu at (0.00, -60.0)
- added J2: , BATTERY_PAD:BATTERY_PAD, F.Cu at (0.00, -390.0)
- added L1: 2.2µH ±20% 750mA 240mΩ, FH_CMH160808B2R2MT:L0603, F.Cu at (0.00, -190.0)
- added L2: 2.2µH ±20% 750mA 240mΩ, FH_CMH160808B2R2MT:L0603, F.Cu at (0.00, -200.0)
- added MK1: , INVENSENSE_MMICT5838_00_012:MIC_T5838, F.Cu at (0.00, -230.0)
- added R10: 0Ω 50mW, UNI_ROYAL_0201WMF0000TEE:R0201, F.Cu at (0.00, -510.0)
- added R11: 33Ω ±5% 50mW, UNI_ROYAL_0201WMJ0330TEE:R0201, F.Cu at (0.00, -520.0)
- added R12: 1MΩ ±1% 50mW, YAGEO_RC0201FR_071ML:R0201, F.Cu at (0.00, -530.0)
- added R13: 47kΩ ±1% 50mW, UNI_ROYAL_0201WMF4702TEE:R0201, F.Cu at (0.00, -540.0)
- added R14: 470kΩ ±1% 50mW, YAGEO_RC0201FR_07470KL:R0201, F.Cu at (0.00, -550.0)
- added R3: 4.7kΩ ±1% 50mW, UNI_ROYAL_0201WMF4701TEE:R0201, F.Cu at (0.00, -440.0)
- added R4: 33Ω ±5% 50mW, UNI_ROYAL_0201WMJ0330TEE:R0201, F.Cu at (0.00, -450.0)
- added R5: 10kΩ ±1% 50mW, UNI_ROYAL_0201WMF1002TEE:R0201, F.Cu at (0.00, -460.0)
- added R6: 10kΩ ±1% 50mW, UNI_ROYAL_0201WMF1002TEE:R0201, F.Cu at (0.00, -470.0)
- added R7: 10kΩ ±1% 50mW, UNI_ROYAL_0201WMF1002TEE:R0201, F.Cu at (0.00, -480.0)
- added R8: 10kΩ ±1% 50mW, UNI_ROYAL_0201WMF1002TEE:R0201, F.Cu at (0.00, -490.0)
- added R9: 10kΩ ±1% 50mW, UNI_ROYAL_0201WMF1002TEE:R0201, F.Cu at (0.00, -500.0)
- added TP1: , POGO_PAD:POGO_PAD, F.Cu at (0.00, -250.0)
- added TP10: , POGO_PAD:POGO_PAD, F.Cu at (0.00, -340.0)
- added TP11: , POGO_PAD:POGO_PAD, F.Cu at (0.00, -350.0)
- added TP12: , POGO_PAD:POGO_PAD, F.Cu at (0.00, -360.0)
- added TP13: , POGO_PAD:POGO_PAD, F.Cu at (0.00, -370.0)
- added TP14: , POGO_PAD:POGO_PAD, F.Cu at (0.00, -400.0)
- added TP2: , POGO_PAD:POGO_PAD, F.Cu at (0.00, -260.0)
- added TP3: , POGO_PAD:POGO_PAD, F.Cu at (0.00, -270.0)
- added TP4: , POGO_PAD:POGO_PAD, F.Cu at (0.00, -280.0)
- added TP5: , POGO_PAD:POGO_PAD, F.Cu at (0.00, -290.0)
- added TP6: , POGO_PAD:POGO_PAD, F.Cu at (0.00, -300.0)
- added TP7: , POGO_PAD:POGO_PAD, F.Cu at (0.00, -310.0)
- added TP8: , POGO_PAD:POGO_PAD, F.Cu at (0.00, -320.0)
- added TP9: , POGO_PAD:POGO_PAD, F.Cu at (0.00, -330.0)
- added U4: , CS_CSNP64GCR01_BOW:LGA-8_L8.5-W7.0-P1.27-TL, F.Cu at (0.00, -240.0)
- added U5: , NORDIC_SEMICONDUCTOR_ASA_nPM1300_QEAA_R7:QFN-32_L5.0-W5.0-P0.50-TL-EP3.5, F.Cu at (0.00, -410.0)
- C1, C2: value 1µF ±10% 25V X5R -> 10µF ±10% 10V X5R; footprint Samsung_Electro_Mechanics_CL05A105KA5NQNC:C0402 -> Samsung_Electro_Mechanics_CL10A106KP8NNNC:C0603
- C3, C4: value 100nF ±10% 16V X7R -> 100nF ±10% X5R; footprint Samsung_Electro_Mechanics_CL05B104KO5NNNC:C0402 -> Murata_Electronics_GRM033R60J104KE19D:C0201
- J1: footprint TYPE_minus_C_minus_31_minus_M_minus_12:USB-C_SMD-TYPE-C-31-M-12_1 -> BATTERY_PAD:BATTERY_PAD
- R1: value 5.1kΩ ±1% 62.5mW -> 0Ω 50mW; footprint UNI_ROYAL_0402WGF5101TCE:R0402 -> UNI_ROYAL_0201WMF0000TEE:R0201
- R2: value 5.1kΩ ±1% 62.5mW -> 4.7kΩ ±1% 50mW; footprint UNI_ROYAL_0402WGF5101TCE:R0402 -> UNI_ROYAL_0201WMF4701TEE:R0201
- U1: footprint USBLC6_minus_2SC6:SOT-23-6_L2.9-W1.6-P0.95-LS2.8-BL -> Texas_Instruments_SN74LVC1T45DPKR:USON-6_L1.6-W1.6-P0.50-BL
- U2: footprint ME6211C33M5G_minus_N:SOT-23-5_L3.0-W1.7-P0.95-LS2.8-BL -> Texas_Instruments_SN74LVC1T45DPKR:USON-6_L1.6-W1.6-P0.50-BL
- U3: footprint E73_minus_2G4M08S1C:WIRELM-SMD_E73-2G4M08S1C -> HJ_N54L_SIP:XCVR_HJ-N54L_SIP
- moved R1 350.0 mm to (0.00, -420.0)
- moved R2 350.0 mm to (0.00, -430.0)
- moved J1 290.0 mm to (0.00, -380.0)
- moved U1 170.0 mm to (0.00, -210.0)
- moved U2 170.0 mm to (0.00, -220.0)
Connections:
- net AI3 renamed P1_11
- net AI4 renamed P2_05
- net NF1 renamed P2_09
- net P0_period_03 renamed P2_10
- net P12 renamed P0_04
- net P1_period_00 renamed P1_09
- net P1_period_02 renamed P2_04
- net P1_period_04 renamed P0_02
- net P1_period_09 renamed P1_12
- net P1_period_11 renamed P0_00
- net P1_period_13 renamed P2_01
- net POGO_I2C_SCL renamed P2_03
- net POGO_I2C_SDA renamed P1_01_NC
- net POGO_RESET renamed P1_00_NC
- net POGO_SWDCLK renamed P1_14
- net POGO_UART_RX renamed P2_08
- net POGO_UART_TX renamed P1_13
- net XL2 renamed P2_02
- C1 pad 1: VBUS -> VCCA
- C2 pad 1: VCC -> VCCB
- C3 pad 1: VCC -> VCCB
- C4 pad 1: VCC -> VCCB
- R1 pad 1: A5 -> RF
- R1 pad 2: GND -> BOARD_ANT
- R2 pad 1: B5 -> SCL
- R2 pad 2: GND -> VCCB
- U1 pad 1: esd-net-0 -> VCCA
- U1 pad 2: esd-net-1 -> GND
- U1 pad 3: esd-net-2 -> footprint-A-0
- U1 pad 4: esd-net-3 -> footprint-B-0
- U1 pad 5: esd-net-4 -> GND
- U1 pad 6: esd-net-5 -> VCCB
- U2 pad 1: VBUS -> VCCA
- U2 pad 3: VBUS -> footprint-A-1
- U2 pad 4: NC -> footprint-B-1
- U2 pad 5: VCC -> VCCA
- U3 pad 10: AI6 -> P1_08
- U3 pad 11: XL1 -> footprint-B-1
- U3 pad 18: AI2 -> P1_10
- U3 pad 19: VCC -> GND
- U3 pad 2: P1_period_10 -> SWDIO
- U3 pad 21: GND -> P2_07
- U3 pad 22: P0_period_07 -> GND
- U3 pad 23: VDH -> RF
- U3 pad 24: GND -> BOARD_ANT
- U3 pad 25: DCH -> GND
- U3 pad 26: ADAPTER_RESET -> SDA
- U3 pad 27: VBS -> SCL
- U3 pad 28: P15 -> SWDCLK
- U3 pad 29: D_minus -> P2_06
- U3 pad 30: P17 -> CMD
- U3 pad 31: D_plus -> P1_15
- U3 pad 33: POGO_SWDIO -> SDDO
- U3 pad 37: ADAPTER_SWDIO -> NRESET
- U3 pad 39: ADAPTER_SWDCLK -> GND
- U3 pad 42: P1_period_06 -> VCCB
- U3 pad 43: NF2 -> VCCB
- U3 pad 5: GND -> P2_00
- U3 pad 7: POGO_3V3_SENSE -> CD_SDD32
- U3 pad 8: AI5 -> P1_02
- U3 pad 9: AI7 -> footprint-B-0

Commit message: wip
Parts:
- R12: value 1MΩ ±1% 50mW -> (none); footprint YAGEO_RC0201FR_071ML:R0201 -> DNP_RES_0201:DNP_RES_0201

Commit message: wip
Parts:
- removed C10, C11, C12, C14, C15, C16, C17, C7, C8, C9: 100nF ±10% X5R, Murata_Electronics_GRM033R60J104KE19D:C0201
- removed C13: 2.2µF ±20% 6.3V X5R, Samsung_Electro_Mechanics_CL05A225MQ5NSNC:C0402
- removed C18, C19, C21: 10µF ±10% 10V X5R, Samsung_Electro_Mechanics_CL10A106KP8NNNC:C0603
- removed C20: 1µF ±10% 25V X5R, Samsung_Electro_Mechanics_CL05A105KA5NQNC:C0402
- removed C5, C6: , DNP_CAP_0201:DNP_CAP_0201
- removed J2: , BATTERY_PAD:BATTERY_PAD
- removed L1, L2: 2.2µH ±20% 750mA 240mΩ, FH_CMH160808B2R2MT:L0603
- removed MK1: , INVENSENSE_MMICT5838_00_012:MIC_T5838
- removed R10: 0Ω 50mW, UNI_ROYAL_0201WMF0000TEE:R0201
- removed R11, R4: 33Ω ±5% 50mW, UNI_ROYAL_0201WMJ0330TEE:R0201
- removed R12: , DNP_RES_0201:DNP_RES_0201
- removed R13: 47kΩ ±1% 50mW, UNI_ROYAL_0201WMF4702TEE:R0201
- removed R14: 470kΩ ±1% 50mW, YAGEO_RC0201FR_07470KL:R0201
- removed R3: 4.7kΩ ±1% 50mW, UNI_ROYAL_0201WMF4701TEE:R0201
- removed R5, R6, R7, R8, R9: 10kΩ ±1% 50mW, UNI_ROYAL_0201WMF1002TEE:R0201
- removed TP13, TP14: , POGO_PAD:POGO_PAD
- removed U4: , CS_CSNP64GCR01_BOW:LGA-8_L8.5-W7.0-P1.27-TL
- removed U5: , NORDIC_SEMICONDUCTOR_ASA_nPM1300_QEAA_R7:QFN-32_L5.0-W5.0-P0.50-TL-EP3.5
- C1, C2: value 10µF ±10% 10V X5R -> 1µF ±10% 25V X5R; footprint Samsung_Electro_Mechanics_CL10A106KP8NNNC:C0603 -> Samsung_Electro_Mechanics_CL05A105KA5NQNC:C0402
- C3, C4: value 100nF ±10% X5R -> 100nF ±10% 16V X7R; footprint Murata_Electronics_GRM033R60J104KE19D:C0201 -> Samsung_Electro_Mechanics_CL05B104KO5NNNC:C0402
- J1: footprint BATTERY_PAD:BATTERY_PAD -> TYPE_minus_C_minus_31_minus_M_minus_12:USB-C_SMD-TYPE-C-31-M-12_1
- R1: value 0Ω 50mW -> 5.1kΩ ±1% 62.5mW; footprint UNI_ROYAL_0201WMF0000TEE:R0201 -> UNI_ROYAL_0402WGF5101TCE:R0402
- R2: value 4.7kΩ ±1% 50mW -> 5.1kΩ ±1% 62.5mW; footprint UNI_ROYAL_0201WMF4701TEE:R0201 -> UNI_ROYAL_0402WGF5101TCE:R0402
- U1: footprint Texas_Instruments_SN74LVC1T45DPKR:USON-6_L1.6-W1.6-P0.50-BL -> USBLC6_minus_2SC6:SOT-23-6_L2.9-W1.6-P0.95-LS2.8-BL
- U2: footprint Texas_Instruments_SN74LVC1T45DPKR:USON-6_L1.6-W1.6-P0.50-BL -> ME6211C33M5G_minus_N:SOT-23-5_L3.0-W1.7-P0.95-LS2.8-BL
- U3: footprint HJ_N54L_SIP:XCVR_HJ-N54L_SIP -> E73_minus_2G4M08S1C:WIRELM-SMD_E73-2G4M08S1C
- moved R1 230.0 mm to (0.00, -190.0)
- moved R2 230.0 mm to (0.00, -200.0)
- moved TP1 180.0 mm to (0.00, -70.0)
- moved TP10 180.0 mm to (0.00, -160.0)
- moved TP11 180.0 mm to (0.00, -170.0)
- moved TP12 180.0 mm to (0.00, -180.0)
- moved TP2 180.0 mm to (0.00, -80.0)
- moved TP3 180.0 mm to (0.00, -90.0)
- moved TP4 180.0 mm to (0.00, -100.0)
- moved TP5 180.0 mm to (0.00, -110.0)
- moved TP6 180.0 mm to (0.00, -120.0)
- moved TP7 180.0 mm to (0.00, -130.0)
- moved TP8 180.0 mm to (0.00, -140.0)
- moved TP9 180.0 mm to (0.00, -150.0)
- moved J1 170.0 mm to (0.00, -210.0)
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Connections:
- net P0_00 renamed P1_period_11
- net P0_02 renamed P1_period_04
- net P0_04 renamed P12
- net P1_09 renamed P1_period_00
- net P1_11 renamed AI3
- net P1_12 renamed P1_period_09
- net P2_01 renamed P1_period_13
- net P2_02 renamed XL2
- net P2_04 renamed P1_period_02
- net P2_05 renamed AI4
- net P2_09 renamed NF1
- net P2_10 renamed P0_period_03
- C1 pad 1: VCCA -> VBUS
- C2 pad 1: VCCB -> VCC
- C3 pad 1: VCCB -> VCC
- C4 pad 1: VCCB -> VCC
- R1 pad 1: RF -> A5
- R1 pad 2: BOARD_ANT -> GND
- R2 pad 1: SCL -> B5
- R2 pad 2: VCCB -> GND
- TP1 pad 1: VCCB -> POGO_3V3_SENSE
- TP10 pad 1: SWDCLK -> POGO_UART_RX
- TP11 pad 1: SWDIO -> POGO_UART_TX
- TP12 pad 1: P1_10 -> VBUS
- TP3 pad 1: SCL -> GND
- TP4 pad 1: SDA -> GND
- TP5 pad 1: SCLK -> POGO_I2C_SCL
- TP6 pad 1: CMD -> POGO_I2C_SDA
- TP7 pad 1: CD_SDD32 -> POGO_RESET
- TP8 pad 1: SDDO -> POGO_SWDCLK
- TP9 pad 1: NRESET -> POGO_SWDIO
- U1 pad 1: VCCA -> esd-net-0
- U1 pad 2: GND -> esd-net-1
- U1 pad 3: footprint-A-0 -> esd-net-2
- U1 pad 4: footprint-B-0 -> esd-net-3
- U1 pad 5: GND -> esd-net-4
- U1 pad 6: VCCB -> esd-net-5
- U2 pad 1: VCCA -> VBUS
- U2 pad 3: footprint-A-1 -> VBUS
- U2 pad 4: footprint-B-1 -> NC
- U2 pad 5: VCCA -> VCC
- U3 pad 10: P1_08 -> AI6
- U3 pad 11: footprint-B-1 -> XL1
- U3 pad 12: P1_01_NC -> POGO_I2C_SDA
- U3 pad 14: P1_13 -> POGO_UART_TX
- U3 pad 16: P2_08 -> POGO_UART_RX
- U3 pad 18: P1_10 -> AI2
- U3 pad 19: GND -> VCC
- U3 pad 2: SWDIO -> P1_period_10
- U3 pad 21: P2_07 -> GND
- U3 pad 22: GND -> P0_period_07
- U3 pad 23: RF -> VDH
- U3 pad 24: BOARD_ANT -> GND
- U3 pad 25: GND -> DCH
- U3 pad 26: SDA -> ADAPTER_RESET
- U3 pad 27: SCL -> VBS
- U3 pad 28: SWDCLK -> P15
- U3 pad 29: P2_06 -> D_minus
- U3 pad 30: CMD -> P17
- U3 pad 31: P1_15 -> D_plus
- U3 pad 32: P1_14 -> POGO_SWDCLK
- U3 pad 33: SDDO -> POGO_SWDIO
- U3 pad 34: P1_00_NC -> POGO_RESET
- U3 pad 35: P2_03 -> POGO_I2C_SCL
- U3 pad 37: NRESET -> ADAPTER_SWDIO
- U3 pad 39: GND -> ADAPTER_SWDCLK
- U3 pad 42: VCCB -> P1_period_06
- U3 pad 43: VCCB -> NF2
- U3 pad 5: P2_00 -> GND
- U3 pad 7: CD_SDD32 -> POGO_3V3_SENSE
- U3 pad 8: P1_02 -> AI5
- U3 pad 9: footprint-B-0 -> AI7

Commit message: wip
Parts:
- added C10: 100nF ±10% X5R, Murata_Electronics_GRM033R60J104KE19D:C0201, F.Cu at (0.00, -70.0)
- added C11: 100nF ±10% X5R, Murata_Electronics_GRM033R60J104KE19D:C0201, F.Cu at (0.00, -80.0)
- added C12: 100nF ±10% X5R, Murata_Electronics_GRM033R60J104KE19D:C0201, F.Cu at (0.00, -90.0)
- added C13: 2.2µF ±20% 6.3V X5R, Samsung_Electro_Mechanics_CL05A225MQ5NSNC:C0402, F.Cu at (0.00, -100.0)
- added C14: 100nF ±10% X5R, Murata_Electronics_GRM033R60J104KE19D:C0201, F.Cu at (0.00, -110.0)
- added C15: 100nF ±10% X5R, Murata_Electronics_GRM033R60J104KE19D:C0201, F.Cu at (0.00, -120.0)
- added C16: 100nF ±10% X5R, Murata_Electronics_GRM033R60J104KE19D:C0201, F.Cu at (0.00, -130.0)
- added C17: 100nF ±10% X5R, Murata_Electronics_GRM033R60J104KE19D:C0201, F.Cu at (0.00, -140.0)
- added C18: 10µF ±10% 10V X5R, Samsung_Electro_Mechanics_CL10A106KP8NNNC:C0603, F.Cu at (0.00, -150.0)
- added C19: 10µF ±10% 10V X5R, Samsung_Electro_Mechanics_CL10A106KP8NNNC:C0603, F.Cu at (0.00, -160.0)
- added C20: 1µF ±10% 25V X5R, Samsung_Electro_Mechanics_CL05A105KA5NQNC:C0402, F.Cu at (0.00, -170.0)
- added C21: 10µF ±10% 10V X5R, Samsung_Electro_Mechanics_CL10A106KP8NNNC:C0603, F.Cu at (0.00, -180.0)
- added C5: , DNP_CAP_0201:DNP_CAP_0201, F.Cu at (0.00, -20.0)
- added C6: , DNP_CAP_0201:DNP_CAP_0201, F.Cu at (0.00, -30.0)
- added C7: 100nF ±10% X5R, Murata_Electronics_GRM033R60J104KE19D:C0201, F.Cu at (0.00, -40.0)
- added C8: 100nF ±10% X5R, Murata_Electronics_GRM033R60J104KE19D:C0201, F.Cu at (0.00, -50.0)
- added C9: 100nF ±10% X5R, Murata_Electronics_GRM033R60J104KE19D:C0201, F.Cu at (0.00, -60.0)
- added J2: , BATTERY_PAD:BATTERY_PAD, F.Cu at (0.00, -390.0)
- added L1: 2.2µH ±20% 750mA 240mΩ, FH_CMH160808B2R2MT:L0603, F.Cu at (0.00, -190.0)
- added L2: 2.2µH ±20% 750mA 240mΩ, FH_CMH160808B2R2MT:L0603, F.Cu at (0.00, -200.0)
- added MK1: , INVENSENSE_MMICT5838_00_012:MIC_T5838, F.Cu at (0.00, -230.0)
- added R10: 0Ω 50mW, UNI_ROYAL_0201WMF0000TEE:R0201, F.Cu at (0.00, -510.0)
- added R11: 33Ω ±5% 50mW, UNI_ROYAL_0201WMJ0330TEE:R0201, F.Cu at (0.00, -520.0)
- added R12: , DNP_RES_0201:DNP_RES_0201, F.Cu at (0.00, -530.0)
- added R13: 47kΩ ±1% 50mW, UNI_ROYAL_0201WMF4702TEE:R0201, F.Cu at (0.00, -540.0)
- added R14: 470kΩ ±1% 50mW, YAGEO_RC0201FR_07470KL:R0201, F.Cu at (0.00, -550.0)
- added R3: 4.7kΩ ±1% 50mW, UNI_ROYAL_0201WMF4701TEE:R0201, F.Cu at (0.00, -440.0)
- added R4: 33Ω ±5% 50mW, UNI_ROYAL_0201WMJ0330TEE:R0201, F.Cu at (0.00, -450.0)
- added R5: 10kΩ ±1% 50mW, UNI_ROYAL_0201WMF1002TEE:R0201, F.Cu at (0.00, -460.0)
- added R6: 10kΩ ±1% 50mW, UNI_ROYAL_0201WMF1002TEE:R0201, F.Cu at (0.00, -470.0)
- added R7: 10kΩ ±1% 50mW, UNI_ROYAL_0201WMF1002TEE:R0201, F.Cu at (0.00, -480.0)
- added R8: 10kΩ ±1% 50mW, UNI_ROYAL_0201WMF1002TEE:R0201, F.Cu at (0.00, -490.0)
- added R9: 10kΩ ±1% 50mW, UNI_ROYAL_0201WMF1002TEE:R0201, F.Cu at (0.00, -500.0)
- added TP13: , POGO_PAD:POGO_PAD, F.Cu at (0.00, -370.0)
- added TP14: , POGO_PAD:POGO_PAD, F.Cu at (0.00, -400.0)
- added U4: , CS_CSNP64GCR01_BOW:LGA-8_L8.5-W7.0-P1.27-TL, F.Cu at (0.00, -240.0)
- added U5: , NORDIC_SEMICONDUCTOR_ASA_nPM1300_QEAA_R7:QFN-32_L5.0-W5.0-P0.50-TL-EP3.5, F.Cu at (0.00, -410.0)
- C1, C2: value 1µF ±10% 25V X5R -> 10µF ±10% 10V X5R; footprint Samsung_Electro_Mechanics_CL05A105KA5NQNC:C0402 -> Samsung_Electro_Mechanics_CL10A106KP8NNNC:C0603
- C3, C4: value 100nF ±10% 16V X7R -> 100nF ±10% X5R; footprint Samsung_Electro_Mechanics_CL05B104KO5NNNC:C0402 -> Murata_Electronics_GRM033R60J104KE19D:C0201
- J1: footprint TYPE_minus_C_minus_31_minus_M_minus_12:USB-C_SMD-TYPE-C-31-M-12_1 -> BATTERY_PAD:BATTERY_PAD
- R1: value 5.1kΩ ±1% 62.5mW -> 0Ω 50mW; footprint UNI_ROYAL_0402WGF5101TCE:R0402 -> UNI_ROYAL_0201WMF0000TEE:R0201
- R2: value 5.1kΩ ±1% 62.5mW -> 4.7kΩ ±1% 50mW; footprint UNI_ROYAL_0402WGF5101TCE:R0402 -> UNI_ROYAL_0201WMF4701TEE:R0201
- U1: footprint USBLC6_minus_2SC6:SOT-23-6_L2.9-W1.6-P0.95-LS2.8-BL -> Texas_Instruments_SN74LVC1T45DPKR:USON-6_L1.6-W1.6-P0.50-BL
- U2: footprint ME6211C33M5G_minus_N:SOT-23-5_L3.0-W1.7-P0.95-LS2.8-BL -> Texas_Instruments_SN74LVC1T45DPKR:USON-6_L1.6-W1.6-P0.50-BL
- U3: footprint E73_minus_2G4M08S1C:WIRELM-SMD_E73-2G4M08S1C -> HJ_N54L_SIP:XCVR_HJ-N54L_SIP
- moved R1 230.0 mm to (0.00, -420.0)
- moved R2 230.0 mm to (0.00, -430.0)
- moved TP1 180.0 mm to (0.00, -250.0)
- moved TP10 180.0 mm to (0.00, -340.0)
- moved TP11 180.0 mm to (0.00, -350.0)
- moved TP12 180.0 mm to (0.00, -360.0)
- moved TP2 180.0 mm to (0.00, -260.0)
- moved TP3 180.0 mm to (0.00, -270.0)
- moved TP4 180.0 mm to (0.00, -280.0)
- moved TP5 180.0 mm to (0.00, -290.0)
- moved TP6 180.0 mm to (0.00, -300.0)
- moved TP7 180.0 mm to (0.00, -310.0)
- moved TP8 180.0 mm to (0.00, -320.0)
- moved TP9 180.0 mm to (0.00, -330.0)
- moved J1 170.0 mm to (0.00, -380.0)
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Connections:
- net AI3 renamed P1_11
- net AI4 renamed P2_05
- net NF1 renamed P2_09
- net P0_period_03 renamed P2_10
- net P12 renamed P0_04
- net P1_period_00 renamed P1_09
- net P1_period_02 renamed P2_04
- net P1_period_04 renamed P0_02
- net P1_period_09 renamed P1_12
- net P1_period_11 renamed P0_00
- net P1_period_13 renamed P2_01
- net XL2 renamed P2_02
- C1 pad 1: VBUS -> VCCA
- C2 pad 1: VCC -> VCCB
- C3 pad 1: VCC -> VCCB
- C4 pad 1: VCC -> VCCB
- R1 pad 1: A5 -> RF
- R1 pad 2: GND -> BOARD_ANT
- R2 pad 1: B5 -> SCL
- R2 pad 2: GND -> VCCB
- TP1 pad 1: POGO_3V3_SENSE -> VCCB
- TP10 pad 1: POGO_UART_RX -> SWDCLK
- TP11 pad 1: POGO_UART_TX -> SWDIO
- TP12 pad 1: VBUS -> P1_10
- TP3 pad 1: GND -> SCL
- TP4 pad 1: GND -> SDA
- TP5 pad 1: POGO_I2C_SCL -> SCLK
- TP6 pad 1: POGO_I2C_SDA -> CMD
- TP7 pad 1: POGO_RESET -> CD_SDD32
- TP8 pad 1: POGO_SWDCLK -> SDDO
- TP9 pad 1: POGO_SWDIO -> NRESET
- U1 pad 1: esd-net-0 -> VCCA
- U1 pad 2: esd-net-1 -> GND
- U1 pad 3: esd-net-2 -> footprint-A-0
- U1 pad 4: esd-net-3 -> footprint-B-0
- U1 pad 5: esd-net-4 -> GND
- U1 pad 6: esd-net-5 -> VCCB
- U2 pad 1: VBUS -> VCCA
- U2 pad 3: VBUS -> footprint-A-1
- U2 pad 4: NC -> footprint-B-1
- U2 pad 5: VCC -> VCCA
- U3 pad 10: AI6 -> P1_08
- U3 pad 11: XL1 -> footprint-B-1
- U3 pad 12: POGO_I2C_SDA -> P1_01_NC
- U3 pad 14: POGO_UART_TX -> P1_13
- U3 pad 16: POGO_UART_RX -> P2_08
- U3 pad 18: AI2 -> P1_10
- U3 pad 19: VCC -> GND
- U3 pad 2: P1_period_10 -> SWDIO
- U3 pad 21: GND -> P2_07
- U3 pad 22: P0_period_07 -> GND
- U3 pad 23: VDH -> RF
- U3 pad 24: GND -> BOARD_ANT
- U3 pad 25: DCH -> GND
- U3 pad 26: ADAPTER_RESET -> SDA
- U3 pad 27: VBS -> SCL
- U3 pad 28: P15 -> SWDCLK
- U3 pad 29: D_minus -> P2_06
- U3 pad 30: P17 -> CMD
- U3 pad 31: D_plus -> P1_15
- U3 pad 32: POGO_SWDCLK -> P1_14
- U3 pad 33: POGO_SWDIO -> SDDO
- U3 pad 34: POGO_RESET -> P1_00_NC
- U3 pad 35: POGO_I2C_SCL -> P2_03
- U3 pad 37: ADAPTER_SWDIO -> NRESET
- U3 pad 39: ADAPTER_SWDCLK -> GND
- U3 pad 42: P1_period_06 -> VCCB
- U3 pad 43: NF2 -> VCCB
- U3 pad 5: GND -> P2_00
- U3 pad 7: POGO_3V3_SENSE -> CD_SDD32
- U3 pad 8: AI5 -> P1_02
- U3 pad 9: AI7 -> footprint-B-0

Commit message: wip
Parts:
- removed C10, C11, C12, C14, C15, C16, C17, C7, C8, C9: 100nF ±10% X5R, Murata_Electronics_GRM033R60J104KE19D:C0201
- removed C13: 2.2µF ±20% 6.3V X5R, Samsung_Electro_Mechanics_CL05A225MQ5NSNC:C0402
- removed C18, C19, C21: 10µF ±10% 10V X5R, Samsung_Electro_Mechanics_CL10A106KP8NNNC:C0603
- removed C20: 1µF ±10% 25V X5R, Samsung_Electro_Mechanics_CL05A105KA5NQNC:C0402
- removed C5, C6: , DNP_CAP_0201:DNP_CAP_0201
- removed J2: , BATTERY_PAD:BATTERY_PAD
- removed L1, L2: 2.2µH ±20% 750mA 240mΩ, FH_CMH160808B2R2MT:L0603
- removed MK1: , INVENSENSE_MMICT5838_00_012:MIC_T5838
- removed R10: 0Ω 50mW, UNI_ROYAL_0201WMF0000TEE:R0201
- removed R11, R4: 33Ω ±5% 50mW, UNI_ROYAL_0201WMJ0330TEE:R0201
- removed R12: , DNP_RES_0201:DNP_RES_0201
- removed R13: 47kΩ ±1% 50mW, UNI_ROYAL_0201WMF4702TEE:R0201
- removed R14: 470kΩ ±1% 50mW, YAGEO_RC0201FR_07470KL:R0201
- removed R3: 4.7kΩ ±1% 50mW, UNI_ROYAL_0201WMF4701TEE:R0201
- removed R5, R6, R7, R8, R9: 10kΩ ±1% 50mW, UNI_ROYAL_0201WMF1002TEE:R0201
- removed TP13, TP14: , POGO_PAD:POGO_PAD
- removed U4: , CS_CSNP64GCR01_BOW:LGA-8_L8.5-W7.0-P1.27-TL
- removed U5: , NORDIC_SEMICONDUCTOR_ASA_nPM1300_QEAA_R7:QFN-32_L5.0-W5.0-P0.50-TL-EP3.5
- C1, C2: value 10µF ±10% 10V X5R -> 1µF ±10% 25V X5R; footprint Samsung_Electro_Mechanics_CL10A106KP8NNNC:C0603 -> Samsung_Electro_Mechanics_CL05A105KA5NQNC:C0402
- C3, C4: value 100nF ±10% X5R -> 100nF ±10% 16V X7R; footprint Murata_Electronics_GRM033R60J104KE19D:C0201 -> Samsung_Electro_Mechanics_CL05B104KO5NNNC:C0402
- J1: footprint BATTERY_PAD:BATTERY_PAD -> TYPE_minus_C_minus_31_minus_M_minus_12:USB-C_SMD-TYPE-C-31-M-12_1
- R1: value 0Ω 50mW -> 5.1kΩ ±1% 62.5mW; footprint UNI_ROYAL_0201WMF0000TEE:R0201 -> UNI_ROYAL_0402WGF5101TCE:R0402
- R2: value 4.7kΩ ±1% 50mW -> 5.1kΩ ±1% 62.5mW; footprint UNI_ROYAL_0201WMF4701TEE:R0201 -> UNI_ROYAL_0402WGF5101TCE:R0402
- U1: footprint Texas_Instruments_SN74LVC1T45DPKR:USON-6_L1.6-W1.6-P0.50-BL -> USBLC6_minus_2SC6:SOT-23-6_L2.9-W1.6-P0.95-LS2.8-BL
- U2: footprint Texas_Instruments_SN74LVC1T45DPKR:USON-6_L1.6-W1.6-P0.50-BL -> ME6211C33M5G_minus_N:SOT-23-5_L3.0-W1.7-P0.95-LS2.8-BL
- U3: footprint HJ_N54L_SIP:XCVR_HJ-N54L_SIP -> E73_minus_2G4M08S1C:WIRELM-SMD_E73-2G4M08S1C
- moved R1 230.0 mm to (0.00, -190.0)
- moved R2 230.0 mm to (0.00, -200.0)
- moved TP1 180.0 mm to (0.00, -70.0)
- moved TP10 180.0 mm to (0.00, -160.0)
- moved TP11 180.0 mm to (0.00, -170.0)
- moved TP12 180.0 mm to (0.00, -180.0)
- moved TP2 180.0 mm to (0.00, -80.0)
- moved TP3 180.0 mm to (0.00, -90.0)
- moved TP4 180.0 mm to (0.00, -100.0)
- moved TP5 180.0 mm to (0.00, -110.0)
- moved TP6 180.0 mm to (0.00, -120.0)
- moved TP7 180.0 mm to (0.00, -130.0)
- moved TP8 180.0 mm to (0.00, -140.0)
- moved TP9 180.0 mm to (0.00, -150.0)
- moved J1 170.0 mm to (0.00, -210.0)
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Connections:
- net P0_00 renamed P1_period_11
- net P0_02 renamed P1_period_04
- net P0_04 renamed P12
- net P1_09 renamed P1_period_00
- net P1_11 renamed AI3
- net P1_12 renamed P1_period_09
- net P2_01 renamed P1_period_13
- net P2_02 renamed XL2
- net P2_04 renamed P1_period_02
- net P2_05 renamed AI4
- net P2_09 renamed NF1
- net P2_10 renamed P0_period_03
- C1 pad 1: VCCA -> VBUS
- C2 pad 1: VCCB -> VCC
- C3 pad 1: VCCB -> VCC
- C4 pad 1: VCCB -> VCC
- R1 pad 1: RF -> A5
- R1 pad 2: BOARD_ANT -> GND
- R2 pad 1: SCL -> B5
- R2 pad 2: VCCB -> GND
- TP1 pad 1: VCCB -> POGO_3V3_SENSE
- TP10 pad 1: SWDCLK -> POGO_UART_RX
- TP11 pad 1: SWDIO -> POGO_UART_TX
- TP12 pad 1: P1_10 -> VBUS
- TP3 pad 1: SCL -> GND
- TP4 pad 1: SDA -> GND
- TP5 pad 1: SCLK -> POGO_I2C_SCL
- TP6 pad 1: CMD -> POGO_I2C_SDA
- TP7 pad 1: CD_SDD32 -> POGO_RESET
- TP8 pad 1: SDDO -> POGO_SWDCLK
- TP9 pad 1: NRESET -> POGO_SWDIO
- U1 pad 1: VCCA -> esd-net-0
- U1 pad 2: GND -> esd-net-1
- U1 pad 3: footprint-A-0 -> esd-net-2
- U1 pad 4: footprint-B-0 -> esd-net-3
- U1 pad 5: GND -> esd-net-4
- U1 pad 6: VCCB -> esd-net-5
- U2 pad 1: VCCA -> VBUS
- U2 pad 3: footprint-A-1 -> VBUS
- U2 pad 4: footprint-B-1 -> NC
- U2 pad 5: VCCA -> VCC
- U3 pad 10: P1_08 -> AI6
- U3 pad 11: footprint-B-1 -> XL1
- U3 pad 12: P1_01_NC -> POGO_I2C_SDA
- U3 pad 14: P1_13 -> POGO_UART_TX
- U3 pad 16: P2_08 -> POGO_UART_RX
- U3 pad 18: P1_10 -> AI2
- U3 pad 19: GND -> VCC
- U3 pad 2: SWDIO -> P1_period_10
- U3 pad 21: P2_07 -> GND
- U3 pad 22: GND -> P0_period_07
- U3 pad 23: RF -> VDH
- U3 pad 24: BOARD_ANT -> GND
- U3 pad 25: GND -> DCH
- U3 pad 26: SDA -> ADAPTER_RESET
- U3 pad 27: SCL -> VBS
- U3 pad 28: SWDCLK -> P15
- U3 pad 29: P2_06 -> D_minus
- U3 pad 30: CMD -> P17
- U3 pad 31: P1_15 -> D_plus
- U3 pad 32: P1_14 -> POGO_SWDCLK
- U3 pad 33: SDDO -> POGO_SWDIO
- U3 pad 34: P1_00_NC -> POGO_RESET
- U3 pad 35: P2_03 -> POGO_I2C_SCL
- U3 pad 37: NRESET -> ADAPTER_SWDIO
- U3 pad 39: GND -> ADAPTER_SWDCLK
- U3 pad 42: VCCB -> P1_period_06
- U3 pad 43: VCCB -> NF2
- U3 pad 5: P2_00 -> GND
- U3 pad 7: CD_SDD32 -> POGO_3V3_SENSE
- U3 pad 8: P1_02 -> AI5
- U3 pad 9: footprint-B-0 -> AI7

Commit message: wip
Connections:
- U3 pad 23: VDH -> VCC
- U3 pad 27: VBS -> VBUS
Changed lines of the file:
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@@
     (net 2 "XL1")
     (net 3 "P1_period_09")
-    (net 4 "VDH")
     (net 5 "A8")
     (net 6 "esd-net-5")
@@
     (net 39 "P1_period_11")
     (net 40 "ADAPTER_SWDCLK")
-    (net 41 "VBS")
     (net 42 "POGO_3V3_SENSE")
     (net 43 "POGO_RESET")
@@
             (size 0.9 2)
             (layers "F.Cu" "F.Paste" "F.Mask")
-            (net 41 "VBS")
+            (net 55 "VBUS")
         )
         (pad "26" smd rect
@@
             (size 0.9 2)
             (layers "F.Cu" "F.Paste" "F.Mask")
-            (net 4 "VDH")
+            (net 35 "VCC")
         )
         (pad "22" smd rect
