File: layouts/main/main.kicad_pcb (KiCad board)
At the start: 4 copper layers, 20 x 20 mm, 60 parts

Commit message: wip
Parts:
- moved L1 257.7 mm to (2.50, -2.30), turned to 90 degrees
- moved U4 1.27 mm to (6.25, -1.25)
Changed lines of the file:
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@@
 	(footprint "NORDIC_SEMICONDUCTOR_ASA_nPM1300_QEAA_R7:QFN-32_L5.0-W5.0-P0.50-TL-EP3.5"
 		(layer "F.Cu")
-		(at 6.5 0)
+		(at 6.25 -1.25)
 		(property "Reference" "U4"
 			(at 0 -6.5 0)
@@
 	(footprint "FH_CMH160808B2R2MT:L0603"
 		(layer "F.Cu")
-		(at 0.27 -260)
+		(at 2.5 -2.3 90)
 		(property "Reference" "L1"
-			(at 0 -4 0)
+			(at 0 -4 90)
 			(layer "F.SilkS")
 			(effects
@@
 		)
 		(property "Value" "2.2µH ±20% 750mA 240mΩ"
-			(at -0.02 0.5 0)
+			(at -0.02 0.5 90)
 			(layer "F.Fab")
 			(effects
@@
 		)
 		(property "Datasheet" "https://wmsc.lcsc.com/wmsc/upload/file/pdf/v2/lcsc/2302231208_FH--Guangdong-Fenghua-Advanced-Tech-CMH160808B2R2MT_C394950.pdf"
-			(at 0 0 0)
+			(at 0 0 90)
 			(layer "User.9")
 			(hide yes)
@@
 		)
 		(property "Description" ""
-			(at 0 0 0)
+			(at 0 0 90)
 			(layer "F.Fab")
 			(hide yes)
@@
 		)
 		(property "checksum" "62ced4c217ba7eae794cd2c7f1cb9ff38caa7cbd67e958863b9b311def40b1ed"
-			(at 0 0 0)
+			(at 0 0 90)
 			(layer "User.9")
 			(hide yes)
@@
 		)
 		(property "__atopile_lib_fp_hash__" "48e12f0b-2e68-eb33-afe4-51b029e84512"
-			(at 0 0 0)
+			(at 0 0 90)
 			(layer "User.9")
 			(hide yes)
@@
 		)
 		(property "LCSC" "C394950"
-			(at 0 0 0)
+			(at 0 0 90)
 			(layer "User.9")
 			(hide yes)
@@
 		)
 		(property "Manufacturer" "FH(Guangdong Fenghua Advanced Tech)"
-			(at 0 0 0)
+			(at 0 0 90)
 			(layer "User.9")
 			(hide yes)
@@
 		)
 		(property "Partnumber" "CMH160808B2R2MT"
-			(at 0 0 0)
+			(at 0 0 90)
 			(layer "User.9")
 			(hide yes)
@@
 		)
 		(property "PARAM_dc_resistance" "{\"type\": \"Quantity_Set_Discrete\", \"data\": {\"intervals\": {\"type\": \"Numeric_Interval_Disjoint\", \"data\": {\"intervals\": [{\"type\": \"Numeric_Interval\", \"data\": {\"min\": 0.24, \"max\": 0.24}}]}}, \"unit\": \"ohm\"}}"
-			(at 0 0 0)
+			(at 0 0 90)
 			(layer "User.9")
 			(hide yes)
@@
 		)
 		(property "PARAM_inductance" "{\"type\": \"Quantity_Interval_Disjoint\", \"data\": {\"intervals\": {\"type\": \"Numeric_Interval_Disjoint\", \"data\": {\"intervals\": [{\"type\": \"Numeric_Interval\", \"data\": {\"min\": 1.759999993e-06, \"max\": 2.640000007e-06}}]}}, \"unit\": \"henry\"}}"
-			(at 0 0 0)
+			(at 0 0 90)
 			(layer "User.9")
 			(hide yes)
@@
 		)
 		(property "PARAM_max_current" "{\"type\": \"Quantity_Set_Discrete\", \"data\": {\"intervals\": {\"type\": \"Numeric_Interval_Disjoint\", \"data\": {\"intervals\": [{\"type\": \"Numeric_Interval\", \"data\": {\"min\": 0.75, \"max\": 0.75}}]}}, \"unit\": \"ampere\"}}"
-			(at 0 0 0)
+			(at 0 0 90)
 			(layer "User.9")
 			(hide yes)
@@
 		)
 		(property "PARAM_saturation_current" "{\"type\": \"Quantity_Interval_Disjoint\", \"data\": {\"intervals\": {\"type\": \"Numeric_Interval_Disjoint\", \"data\": {\"intervals\": [{\"type\": \"Numeric_Interval\", \"data\": {\"min\": 0.0, \"max\": null}}]}}, \"unit\": \"ampere\"}}"
-			(at 0 0 0)
+			(at 0 0 90)
 			(layer "User.9")
 			(hide yes)
@@
 		)
 		(property "PARAM_self_resonant_frequency" "{\"type\": \"Quantity_Interval_Disjoint\", \"data\": {\"intervals\": {\"type\": \"Numeric_Interval_Disjoint\", \"data\": {\"intervals\": [{\"type\": \"Numeric_Interval\", \"data\": {\"min\": 0.0, \"max\": null}}]}}, \"unit\": \"hertz\"}}"
-			(at 0 0 0)
+			(at 0 0 90)
 			(layer "User.9")
 			(hide yes)
@@
 		)
 		(property "atopile_address" "l_buck1"
-			(at 0 0 0)
+			(at 0 0 90)
 			(layer "User.9")
 			(hide yes)
@@
 		(attr smd)
 		(fp_line
-			(start -1.43 -0.51)
-			(end -1.27 -0.65)
+			(start 1.27 -0.65)
+			(end 0.51 -0.65)
 			(stroke
 				(width 0.15)
@@
 		)
 		(fp_line
-			(start -1.43 0.5)
-			(end -1.43 -0.51)
+			(start 1.27 -0.65)
+			(end 1.42 -0.5)
 			(stroke
 				(width 0.15)
@@
 		)
 		(fp_line
-			(start -1.28 0.65)
-			(end -0.51 0.65)
+			(start -1.43 -0.51)
+			(end -1.27 -0.65)
 			(stroke
 				(width 0.15)
@@
 		)
 		(fp_line
-			(start -1.27 0.65)
-			(end -1.43 0.5)
+			(start 1.42 -0.5)
+			(end 1.42 0.52)
 			(stroke
 				(width 0.15)
@@
 		)
 		(fp_line
-			(start 1.27 -0.65)
-			(end 0.51 -0.65)
+			(start -1.43 0.5)
+			(end -1.43 -0.51)
 			(stroke
 				(width 0.15)
@@
 		)
 		(fp_line
-			(start 1.27 -0.65)
-			(end 1.42 -0.5)
+			(start 1.42 0.52)
+			(end 1.27 0.65)
 			(stroke
 				(width 0.15)
@@
 		)
 		(fp_line
-			(start 1.42 -0.5)
-			(end 1.42 0.52)
+			(start -1.27 0.65)
+			(end -1.43 0.5)
 			(stroke
 				(width 0.15)
@@
 		)
 		(fp_line
-			(start 1.42 0.52)
-			(end 1.27 0.65)
+			(start -1.28 0.65)
+			(end -0.51 0.65)
 			(stroke
 				(width 0.15)
@@
 		)
 		(fp_text user "${REFERENCE}"
-			(at 0 -4 0)
+			(at 0 -4 90)
 			(layer "F.SilkS")
 			(effects
@@
 		)
 		(fp_text user "${REFERENCE}"
-			(at 0 -0.5 0)
+			(at 0 -0.5 90)
 			(layer "F.Fab")
 			(effects
@@
 		)
 		(pad "1" smd rect
-			(at -0.7 0 180)
+			(at -0.7 0 270)
 			(size 0.8 0.86)
 			(layers "F.Cu" "F.Mask" "F.Paste")
@@
 		)
 		(pad "2" smd rect
-			(at 0.7 0 180)
+			(at 0.7 0 270)
 			(size 0.8 0.86)
 			(layers "F.Cu" "F.Mask" "F.Paste")
@@
 		)
 		(property "Value" "XCVR_HJ-N54L_SIP"
-			(at 1.875 -3.525 0)
+			(at 2.875 -3.525 0)
 			(layer "F.Fab")
 			(effects

Commit message: wip
Parts:
- moved R14 633.8 mm to (5.75, 3.74), turned to -90 degrees
- moved R13 623.0 mm to (6.75, 2.99), turned to -90 degrees
- moved L2 270.8 mm to (-0.45, 0.75), turned to 180 degrees
- moved C22 248.1 mm to (8.75, -2.05), turned to 90 degrees
- moved C21 244.0 mm to (4.50, 3.92), turned to -90 degrees
- moved C20 228.3 mm to (7.75, -1.83), turned to 90 degrees
- moved C19 221.2 mm to (8.70, 1.00)
- moved C18 212.4 mm to (8.45, 2.25)
- moved C17 199.4 mm to (8.02, -0.75)
- moved C16 190.2 mm to (7.92, 0.00)
- moved C15 176.6 mm to (6.27, -3.50)
- moved C14 166.8 mm to (2.02, -3.25)
- moved C13 163.8 mm to (3.75, 3.77), turned to -90 degrees
- moved C12 149.8 mm to (9.27, -0.50)
- moved R10 81.2 mm to (7.49, 3.25)
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
Commit message: wip
Parts:
- moved REF** 486.5 mm to (6.25, 6.50)
- moved REF** 473.6 mm to (8.50, 3.50)
- moved REF** 467.8 mm to (2.75, 7.75)
- moved REF** 455.8 mm to (4.25, 5.75), turned to -90 degrees
- moved REF** 407.8 mm to (4.75, 7.75)
- moved REF** 325.1 mm to (7.75, 5.00)
- moved C7 1.27 mm to (-0.02, -9.25)
- moved C15 0.54 mm to (6.48, -3.00)
- moved C14 0.25 mm to (2.02, -3.00)
- moved C2 0.25 mm to (4.45, -3.50)
- moved REF** 0.25 mm to (0.00, -9.75)
Changed lines of the file:
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@@
 	(footprint "POGO_PAD:POGO_PAD"
 		(layer "F.Cu")
-		(at 0.27 -320)
+		(at 7.75 5)
 		(property "Reference" "REF**"
 			(at 0 -1.5 0)
@@
 	(footprint "POGO_PAD:POGO_PAD"
 		(layer "F.Cu")
-		(at 0.27 -400)
+		(at 4.75 7.75)
 		(property "Reference" "REF**"
 			(at 0 -1.5 0)
@@
 	(footprint "POGO_PAD:POGO_PAD"
 		(layer "F.Cu")
-		(at 0.27 -470)
+		(at 8.5 3.5)
 		(property "Reference" "REF**"
 			(at 0 -1.5 0)
@@
 	(footprint "Murata_Electronics_GRM033R60J104KE19D:C0201"
 		(layer "F.Cu")
-		(at 2.02 -3.25)
+		(at 2.02 -3)
 		(property "Reference" "C14"
 			(at 0 -4 0)
@@
 	(footprint "BATTERY_PAD:BATTERY_PAD"
 		(layer "F.Cu")
-		(at 0.27 -450)
+		(at 4.25 5.75 -90)
 		(property "Reference" "REF**"
-			(at 0 -2 0)
+			(at 0 -2 90)
 			(layer "F.SilkS")
 			(effects
@@
 		)
 		(property "Value" "BATTERY_PAD"
-			(at 0 1.25 0)
+			(at 0 1.25 90)
 			(layer "F.Fab")
 			(effects
@@
 		)
 		(property "Datasheet" ""
-			(at 0 0 0)
+			(at 0 0 90)
 			(layer "F.Fab")
 			(hide yes)
@@
 		)
 		(property "Description" ""
-			(at 0 0 0)
+			(at 0 0 90)
 			(layer "F.Fab")
 			(hide yes)
@@
 		)
 		(property "__atopile_lib_fp_hash__" "1ac2203b-ca3b-6f6f-d097-7eae861b36bf"
-			(at 0 0 0)
+			(at 0 0 90)
 			(layer "User.9")
 			(hide yes)
@@
 		)
 		(property "atopile_address" "pad_vbat_n"
-			(at 0 0 0)
+			(at 0 0 90)
 			(layer "User.9")
 			(hide yes)
@@
 		(attr smd)
 		(fp_line
-			(start -1 -1.25)
-			(end -1 1.25)
+			(start -1 1.25)
+			(end 1 1.25)
 			(stroke
 				(width 0.12)
@@
 		(fp_line
 			(start -1 -1.25)
-			(end 1 -1.25)
+			(end -1 1.25)
 			(stroke
 				(width 0.12)
@@
 		)
 		(fp_line
-			(start -1 1.25)
-			(end 1 1.25)
+			(start -1 -1.25)
+			(end 1 -1.25)
 			(stroke
 				(width 0.12)
@@
 		)
 		(fp_line
-			(start -1.2 -1.45)
-			(end -1.2 1.45)
+			(start -1.2 1.45)
+			(end 1.2 1.45)
 			(stroke
 				(width 0.05)
@@
 		(fp_line
 			(start -1.2 -1.45)
-			(end 1.2 -1.45)
+			(end -1.2 1.45)
 			(stroke
 				(width 0.05)
@@
 		)
 		(fp_line
-			(start -1.2 1.45)
-			(end 1.2 1.45)
+			(start -1.2 -1.45)
+			(end 1.2 -1.45)
 			(stroke
 				(width 0.05)
@@
 		)
 		(pad "1" smd rect
-			(at 0 0)
+			(at 0 0 270)
 			(size 1.5 2)
 			(layers "F.Cu" "F.Mask" "F.Paste")
@@
 	(footprint "Samsung_Electro_Mechanics_CL10A106KP8NNNC:C0603"
 		(layer "F.Cu")
-		(at 4.45 -3.75)
+		(at 4.45 -3.5)
 		(property "Reference" "C2"
 			(at 0 -4 0)
@@
 	(footprint "Murata_Electronics_GRM033R60J104KE19D:C0201"
 		(layer "F.Cu")
-		(at 6.27 -3.5)
+		(at 6.48 -3)
 		(property "Reference" "C15"
 			(at 0 -4 0)
@@
 	(footprint "DNP_CAP_0201:DNP_CAP_0201"
 		(layer "F.Cu")
-		(at 0 -9.5)
+		(at 0 -9.75)
 		(property "Reference" "REF**"
 			(at 0 -1.1 0)
@@
 	(footprint "POGO_PAD:POGO_PAD"
 		(layer "F.Cu")
-		(at 0.27 -480)
+		(at 6.25 6.5)
 		(property "Reference" "REF**"
 			(at 0 -1.5 0)
@@
 	(footprint "Murata_Electronics_GRM033R60J104KE19D:C0201"
 		(layer "F.Cu")
-		(at -1.27 -9.5)
+		(at -0.02 -9.25)
 		(property "Reference" "C7"
 			(at 0 -4 0)
@@
 	(footprint "BATTERY_PAD:BATTERY_PAD"
 		(layer "F.Cu")
-		(at 0.27 -460)
+		(at 2.75 7.75)
 		(property "Reference" "REF**"
 			(at 0 -2 0)

Commit message: wip
Parts:
- moved C1 1.35 mm to (0.05, -3.00)
- moved L2 0.83 mm to (0.00, 1.45), turned to -90 degrees
- moved L1 0.71 mm to (0.00, -1.05), turned to 90 degrees

Commit message: wip
Parts:
- moved R7 565.3 mm to (-4.75, 5.24), turned to -90 degrees
- moved R6 555.3 mm to (-6.00, 5.25), turned to -90 degrees
- moved R5 545.3 mm to (-7.25, 5.24), turned to -90 degrees
- moved R4 526.0 mm to (-0.50, -4.00), turned to 90 degrees
- moved U3 310.3 mm to (-5.68, 0.24), turned to -90 degrees
- moved REF** 307.3 mm to (1.48, 7.29)
- moved U1 287.7 mm to (-2.73, 7.70)
- moved C11 143.9 mm to (0.33, 3.92), turned to 90 degrees
- moved C10 134.0 mm to (-0.75, 4.02), turned to 90 degrees
- moved REF** 14.2 mm to (5.25, -6.25), turned to -90 degrees
- moved REF** 10.7 mm to (7.25, -4.50), turned to 180 degrees
- moved REF** 3.26 mm to (6.50, 5.00)
- moved L2 0.43 mm to (0.25, 1.80)
- moved L1 0.27 mm to (0.25, -0.95)
- moved C1 0.25 mm to (0.05, -2.75)

Commit message: wip
Parts:
- moved R9 575.0 mm to (-4.49, -5.00), turned to 90 degrees
- moved R8 565.0 mm to (-3.25, -5.00), turned to 90 degrees
- moved REF** 373.5 mm to (-4.75, -6.50)
- moved REF** 363.5 mm to (-3.00, -6.50)
- moved REF** 355.1 mm to (-7.50, -5.00)
- moved REF** 344.8 mm to (-6.00, -5.25)
- moved REF** 0.90 mm to (7.00, 6.00)
- moved REF** 0.25 mm to (7.75, 4.75)
- moved REF** 0.25 mm to (6.50, 4.75)
Changed lines of the file:
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@@
 	(footprint "POGO_PAD:POGO_PAD"
 		(layer "F.Cu")
-		(at 0.27 -360)
+		(at -7.5 -5)
 		(property "Reference" "REF**"
 			(at 0 -1.5 0)
@@
 	(footprint "POGO_PAD:POGO_PAD"
 		(layer "F.Cu")
-		(at 7.75 5)
+		(at 7.75 4.75)
 		(property "Reference" "REF**"
 			(at 0 -1.5 0)
@@
 	(footprint "UNI_ROYAL_0201WMF1002TEE:R0201"
 		(layer "F.Cu")
-		(at 0.27 -570)
+		(at -3.25 -5 90)
 		(property "Reference" "R8"
-			(at 0 -4 0)
+			(at 0 -4 90)
 			(layer "F.SilkS")
 			(effects
@@
 		)
 		(property "Value" "10kΩ ±1% 50mW"
-			(at 0 0.25 0)
+			(at 0 0.25 90)
 			(layer "F.Fab")
 			(effects
@@
 		)
 		(property "Datasheet" "https://wmsc.lcsc.com/wmsc/upload/file/pdf/v2/lcsc/2205312145_UNI-ROYAL-Uniroyal-Elec-0201WMF1002TEE_C473048.pdf"
-			(at 0 0 0)
+			(at 0 0 90)
 			(layer "User.9")
 			(hide yes)
@@
 		)
 		(property "Description" ""
-			(at 0 0 0)
+			(at 0 0 90)
 			(layer "F.Fab")
 			(hide yes)
@@
 		)
 		(property "checksum" "d54b648b29e4db75dc4a06617f8364f1a2000b36bd119b9bd4dbb9f90bd7bcfc"
-			(at 0 0 0)
+			(at 0 0 90)
 			(layer "User.9")
 			(hide yes)
@@
 		)
 		(property "__atopile_lib_fp_hash__" "fb4bc967-e06e-5b83-c2ec-7df19a197edb"
-			(at 0 0 0)
+			(at 0 0 90)
 			(layer "User.9")
 			(hide yes)
@@
 		)
 		(property "LCSC" "C473048"
-			(at 0 0 0)
+			(at 0 0 90)
 			(layer "User.9")
 			(hide yes)
@@
 		)
 		(property "Manufacturer" "UNI-ROYAL(Uniroyal Elec)"
-			(at 0 0 0)
+			(at 0 0 90)
 			(layer "User.9")
 			(hide yes)
@@
 		)
 		(property "Partnumber" "0201WMF1002TEE"
-			(at 0 0 0)
+			(at 0 0 90)
 			(layer "User.9")
 			(hide yes)
@@
 		)
 		(property "PARAM_max_power" "{\"type\": \"Quantity_Set_Discrete\", \"data\": {\"intervals\": {\"type\": \"Numeric_Interval_Disjoint\", \"data\": {\"intervals\": [{\"type\": \"Numeric_Interval\", \"data\": {\"min\": 0.05, \"max\": 0.05}}]}}, \"unit\": \"watt\"}}"
-			(at 0 0 0)
+			(at 0 0 90)
 			(layer "User.9")
 			(hide yes)
@@
 		)
 		(property "PARAM_max_voltage" "{\"type\": \"Quantity_Set_Discrete\", \"data\": {\"intervals\": {\"type\": \"Numeric_Interval_Disjoint\", \"data\": {\"intervals\": [{\"type\": \"Numeric_Interval\", \"data\": {\"min\": 25.0, \"max\": 25.0}}]}}, \"unit\": \"volt\"}}"
-			(at 0 0 0)
+			(at 0 0 90)
 			(layer "User.9")
 			(hide yes)
@@
 		)
 		(property "PARAM_resistance" "{\"type\": \"Quantity_Interval_Disjoint\", \"data\": {\"intervals\": {\"type\": \"Numeric_Interval_Disjoint\", \"data\": {\"intervals\": [{\"type\": \"Numeric_Interval\", \"data\": {\"min\": 9900.000002235174, \"max\": 10099.999997764826}}]}}, \"unit\": \"ohm\"}}"
-			(at 0 0 0)
+			(at 0 0 90)
 			(layer "User.9")
 			(hide yes)
@@
 		)
 		(property "atopile_address" "r_nand_dat2"
-			(at 0 0 0)
+			(at 0 0 90)
 			(layer "User.9")
 			(hide yes)
@@
 		(attr through_hole)
 		(fp_line
-			(start -0.62 -0.39)
-			(end -0.17 -0.39)
+			(start 0.62 -0.39)
+			(end 0.17 -0.39)
 			(stroke
 				(width 0.15)
@@
 		)
 		(fp_line
-			(start -0.62 0.39)
-			(end -0.62 -0.39)
+			(start -0.62 -0.39)
+			(end -0.17 -0.39)
 			(stroke
 				(width 0.15)
@@
 		)
 		(fp_line
-			(start -0.17 0.39)
-			(end -0.62 0.39)
+			(start 0.62 0.39)
+			(end 0.62 -0.39)
 			(stroke
 				(width 0.15)
@@
 		)
 		(fp_line
-			(start 0.62 -0.39)
-			(end 0.17 -0.39)
+			(start -0.17 0.39)
+			(end -0.62 0.39)
 			(stroke
 				(width 0.15)
@@
 		)
 		(fp_line
-			(start 0.62 0.39)
-			(end 0.62 -0.39)
+			(start -0.62 0.39)
+			(end -0.62 -0.39)
 			(stroke
 				(width 0.15)
@@
 		)
 		(fp_text user "${REFERENCE}"
-			(at 0 -4 0)
+			(at 0 -4 90)
 			(layer "F.SilkS")
 			(effects
@@
 		)
 		(fp_text user "${REFERENCE}"
-			(at 0 -0.25 0)
+			(at 0 -0.25 90)
 			(layer "F.Fab")
 			(effects
@@
 		)
 		(pad "1" smd rect
-			(at -0.24 0)
+			(at -0.24 0 90)
 			(size 0.3 0.32)
 			(layers "F.Cu" "F.Mask" "F.Paste")
@@
 		)
 		(pad "2" smd rect
-			(at 0.24 0)
+			(at 0.24 0 90)
 			(size 0.3 0.32)
 			(layers "F.Cu" "F.Mask" "F.Paste")
@@
 	(footprint "POGO_PAD:POGO_PAD"
 		(layer "F.Cu")
-		(at 0.27 -350)
+		(at -6 -5.25)
 		(property "Reference" "REF**"
 			(at 0 -1.5 0)
@@
 	(footprint "POGO_PAD:POGO_PAD"
 		(layer "F.Cu")
-		(at 6.5 5)
+		(at 6.5 4.75)
 		(property "Reference" "REF**"
 			(at 0 -1.5 0)
@@
 	(footprint "POGO_PAD:POGO_PAD"
 		(layer "F.Cu")
-		(at 0.27 -370)
+		(at -3 -6.5)
 		(property "Reference" "REF**"
 			(at 0 -1.5 0)
@@
 	(footprint "POGO_PAD:POGO_PAD"
 		(layer "F.Cu")
-		(at 0.27 -380)
+		(at -4.75 -6.5)
 		(property "Reference" "REF**"
 			(at 0 -1.5 0)
@@
 	(footprint "POGO_PAD:POGO_PAD"
 		(layer "F.Cu")
-		(at 6.25 6.5)
+		(at 7 6)
 		(property "Reference" "REF**"
 			(at 0 -1.5 0)
@@
 	(footprint "UNI_ROYAL_0201WMF1002TEE:R0201"
 		(layer "F.Cu")
-		(at 0.27 -580)
+		(at -4.49 -5 90)
 		(property "Reference" "R9"
-			(at 0 -4 0)
+			(at 0 -4 90)
 			(layer "F.SilkS")
 			(effects
@@
 		)
 		(property "Value" "10kΩ ±1% 50mW"
-			(at -0.02 0.25 0)
+			(at -0.02 0.25 90)
 			(layer "F.Fab")
 			(effects
@@
 		)
 		(property "Datasheet" "https://wmsc.lcsc.com/wmsc/upload/file/pdf/v2/lcsc/2205312145_UNI-ROYAL-Uniroyal-Elec-0201WMF1002TEE_C473048.pdf"
-			(at 0 0 0)
+			(at 0 0 90)
 			(layer "User.9")
 			(hide yes)
@@
 		)
 		(property "Description" ""
-			(at 0 0 0)
+			(at 0 0 90)
 			(layer "F.Fab")
 			(hide yes)
@@
 		)
 		(property "checksum" "d54b648b29e4db75dc4a06617f8364f1a2000b36bd119b9bd4dbb9f90bd7bcfc"
-			(at 0 0 0)
+			(at 0 0 90)
 			(layer "User.9")
 			(hide yes)
@@
 		)
 		(property "__atopile_lib_fp_hash__" "fb4bc967-e06e-5b83-c2ec-7df19a197edb"
-			(at 0 0 0)
+			(at 0 0 90)
 			(layer "User.9")
 			(hide yes)
@@
 		)
 		(property "LCSC" "C473048"
-			(at 0 0 0)
+			(at 0 0 90)
 			(layer "User.9")
 			(hide yes)
@@
 		)
 		(property "Manufacturer" "UNI-ROYAL(Uniroyal Elec)"
-			(at 0 0 0)
+			(at 0 0 90)
 			(layer "User.9")
 			(hide yes)
@@
 		)
 		(property "Partnumber" "0201WMF1002TEE"
-			(at 0 0 0)
+			(at 0 0 90)
 			(layer "User.9")
 			(hide yes)
@@
 		)
 		(property "PARAM_max_power" "{\"type\": \"Quantity_Set_Discrete\", \"data\": {\"intervals\": {\"type\": \"Numeric_Interval_Disjoint\", \"data\": {\"intervals\": [{\"type\": \"Numeric_Interval\", \"data\": {\"min\": 0.05, \"max\": 0.05}}]}}, \"unit\": \"watt\"}}"
-			(at 0 0 0)
+			(at 0 0 90)
 			(layer "User.9")
 			(hide yes)
@@
 		)
 		(property "PARAM_max_voltage" "{\"type\": \"Quantity_Set_Discrete\", \"data\": {\"intervals\": {\"type\": \"Numeric_Interval_Disjoint\", \"data\": {\"intervals\": [{\"type\": \"Numeric_Interval\", \"data\": {\"min\": 25.0, \"max\": 25.0}}]}}, \"unit\": \"volt\"}}"
-			(at 0 0 0)
+			(at 0 0 90)
 			(layer "User.9")
 			(hide yes)
@@
 		)
 		(property "PARAM_resistance" "{\"type\": \"Quantity_Interval_Disjoint\", \"data\": {\"intervals\": {\"type\": \"Numeric_Interval_Disjoint\", \"data\": {\"intervals\": [{\"type\": \"Numeric_Interval\", \"data\": {\"min\": 9900.000002235174, \"max\": 10099.999997764826}}]}}, \"unit\": \"ohm\"}}"
-			(at 0 0 0)
+			(at 0 0 90)
 			(layer "User.9")
 			(hide yes)
@@
 		)
 		(property "atopile_address" "r_nand_dat3"
-			(at 0 0 0)
+			(at 0 0 90)
 			(layer "User.9")
 			(hide yes)
@@
 		(attr through_hole)
 		(fp_line
-			(start -0.62 -0.39)
-			(end -0.17 -0.39)
+			(start 0.62 -0.39)
+			(end 0.17 -0.39)
 			(stroke
 				(width 0.15)
@@
 		)
 		(fp_line
-			(start -0.62 0.39)
-			(end -0.62 -0.39)
+			(start -0.62 -0.39)
+			(end -0.17 -0.39)
 			(stroke
 				(width 0.15)
@@
 		)
 		(fp_line
-			(start -0.17 0.39)
-			(end -0.62 0.39)
+			(start 0.62 0.39)
+			(end 0.62 -0.39)
 			(stroke
 				(width 0.15)
@@
 		)
 		(fp_line
-			(start 0.62 -0.39)
-			(end 0.17 -0.39)
+			(start -0.17 0.39)
+			(end -0.62 0.39)
 			(stroke
 				(width 0.15)
@@
 		)
 		(fp_line
-			(start 0.62 0.39)
-			(end 0.62 -0.39)
+			(start -0.62 0.39)
+			(end -0.62 -0.39)
 			(stroke
 				(width 0.15)
@@
 		)
 		(fp_text user "${REFERENCE}"
-			(at 0 -4 0)
+			(at 0 -4 90)
 			(layer "F.SilkS")
 			(effects
@@
 		)
 		(fp_text user "${REFERENCE}"
-			(at 0 -0.25 0)
+			(at 0 -0.25 90)
 			(layer "F.Fab")
 			(effects
@@
 		)
 		(pad "1" smd rect
-			(at -0.24 0)
+			(at -0.24 0 90)
 			(size 0.3 0.32)
 			(layers "F.Cu" "F.Mask" "F.Paste")
@@
 		)
 		(pad "2" smd rect
-			(at 0.24 0)
+			(at 0.24 0 90)
 			(size 0.3 0.32)
 			(layers "F.Cu" "F.Mask" "F.Paste")

Commit message: wip
Parts:
- moved REF** 618.3 mm to (-0.57, 8.25)
- moved R11 609.3 mm to (-0.74, 9.25)
- moved C9 125.8 mm to (4.00, 5.77), turned to 90 degrees
- moved C6 98.1 mm to (-4.73, 8.00), turned to 180 degrees
- moved C5 85.3 mm to (-2.48, 5.25)
- moved REF** 0.44 mm to (1.91, 7.29)
- moved U1 0.35 mm to (-2.70, 7.35), turned to 90 degrees
