File: layouts/main/main.kicad_pcb (KiCad board)
At the start: 4 copper layers, 20 x 20 mm, 60 parts

Commit message: wip
Parts:
- moved R3 515.2 mm to (-2.50, -4.76), turned to -90 degrees
- moved R2 506.3 mm to (-1.49, -3.75)
- moved REF** 431.4 mm to (-12.5, -8.75)
- moved REF** 425.4 mm to (-11.8, -4.75)
- moved REF** 418.4 mm to (-11.8, -1.75)
- moved REF** 411.9 mm to (-11.0, 1.75)
- moved REF** 395.2 mm to (-10.8, 5.00)
- moved REF** 348.2 mm to (-10.2, 8.00)
- moved REF** 341.2 mm to (-10.5, 11.0)
- moved R8 0.25 mm to (-3.50, -5.00)
Changed lines of the file:
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@@
 	(footprint "UNI_ROYAL_0201WMF1002TEE:R0201"
 		(layer "F.Cu")
-		(at -3.25 -5 90)
+		(at -3.5 -5 90)
 		(property "Reference" "R8"
 			(at 0 -4 90)
@@
 	(footprint "POGO_PAD:POGO_PAD"
 		(layer "F.Cu")
-		(at 0.27 -340)
+		(at -10.25 8)
 		(property "Reference" "REF**"
 			(at 0 -1.5 0)
@@
 	(footprint "POGO_PAD:POGO_PAD"
 		(layer "F.Cu")
-		(at 0.27 -410)
+		(at -11 1.75)
 		(property "Reference" "REF**"
 			(at 0 -1.5 0)
@@
 	(footprint "UNI_ROYAL_0201WMF4701TEE:R0201"
 		(layer "F.Cu")
-		(at 0.27 -520)
+		(at -2.5 -4.76 -90)
 		(property "Reference" "R3"
-			(at 0 -4 0)
+			(at 0 -4 90)
 			(layer "F.SilkS")
 			(effects
@@
 		)
 		(property "Value" "4.7kΩ ±1% 50mW"
-			(at 0 0.25 0)
+			(at 0 0.25 90)
 			(layer "F.Fab")
 			(effects
@@
 		)
 		(property "Datasheet" "https://wmsc.lcsc.com/wmsc/upload/file/pdf/v2/lcsc/2205311945_UNI-ROYAL-Uniroyal-Elec-0201WMF4701TEE_C270346.pdf"
-			(at 0 0 0)
+			(at 0 0 90)
 			(layer "User.9")
 			(hide yes)
@@
 		)
 		(property "Description" ""
-			(at 0 0 0)
+			(at 0 0 90)
 			(layer "F.Fab")
 			(hide yes)
@@
 		)
 		(property "checksum" "8334129e8d68cc94feb6f24d4494287d4e5c79980c878904c53191d3ecd9f05e"
-			(at 0 0 0)
+			(at 0 0 90)
 			(layer "User.9")
 			(hide yes)
@@
 		)
 		(property "__atopile_lib_fp_hash__" "d667899d-2d9d-7d5e-0a90-0fa71e28edb2"
-			(at 0 0 0)
+			(at 0 0 90)
 			(layer "User.9")
 			(hide yes)
@@
 		)
 		(property "LCSC" "C270346"
-			(at 0 0 0)
+			(at 0 0 90)
 			(layer "User.9")
 			(hide yes)
@@
 		)
 		(property "Manufacturer" "UNI-ROYAL(Uniroyal Elec)"
-			(at 0 0 0)
+			(at 0 0 90)
 			(layer "User.9")
 			(hide yes)
@@
 		)
 		(property "Partnumber" "0201WMF4701TEE"
-			(at 0 0 0)
+			(at 0 0 90)
 			(layer "User.9")
 			(hide yes)
@@
 		)
 		(property "PARAM_max_power" "{\"type\": \"Quantity_Set_Discrete\", \"data\": {\"intervals\": {\"type\": \"Numeric_Interval_Disjoint\", \"data\": {\"intervals\": [{\"type\": \"Numeric_Interval\", \"data\": {\"min\": 0.05, \"max\": 0.05}}]}}, \"unit\": \"watt\"}}"
-			(at 0 0 0)
+			(at 0 0 90)
 			(layer "User.9")
 			(hide yes)
@@
 		)
 		(property "PARAM_max_voltage" "{\"type\": \"Quantity_Set_Discrete\", \"data\": {\"intervals\": {\"type\": \"Numeric_Interval_Disjoint\", \"data\": {\"intervals\": [{\"type\": \"Numeric_Interval\", \"data\": {\"min\": 25.0, \"max\": 25.0}}]}}, \"unit\": \"volt\"}}"
-			(at 0 0 0)
+			(at 0 0 90)
 			(layer "User.9")
 			(hide yes)
@@
 		)
 		(property "PARAM_resistance" "{\"type\": \"Quantity_Interval_Disjoint\", \"data\": {\"intervals\": {\"type\": \"Numeric_Interval_Disjoint\", \"data\": {\"intervals\": [{\"type\": \"Numeric_Interval\", \"data\": {\"min\": 4653.000001050532, \"max\": 4746.999998949468}}]}}, \"unit\": \"ohm\"}}"
-			(at 0 0 0)
+			(at 0 0 90)
 			(layer "User.9")
 			(hide yes)
@@
 		)
 		(property "atopile_address" "r_i2c_sda"
-			(at 0 0 0)
+			(at 0 0 90)
 			(layer "User.9")
 			(hide yes)
@@
 		(attr through_hole)
 		(fp_line
-			(start -0.62 -0.39)
-			(end -0.17 -0.39)
+			(start -0.62 0.39)
+			(end -0.62 -0.39)
 			(stroke
 				(width 0.15)
@@
 		)
 		(fp_line
-			(start -0.62 0.39)
-			(end -0.62 -0.39)
+			(start -0.17 0.39)
+			(end -0.62 0.39)
 			(stroke
 				(width 0.15)
@@
 		)
 		(fp_line
-			(start -0.17 0.39)
-			(end -0.62 0.39)
+			(start 0.17 0.39)
+			(end 0.62 0.39)
 			(stroke
 				(width 0.15)
@@
 		)
 		(fp_line
-			(start 0.17 0.39)
-			(end 0.62 0.39)
+			(start 0.62 0.39)
+			(end 0.62 -0.39)
 			(stroke
 				(width 0.15)
@@
 		)
 		(fp_line
-			(start 0.62 -0.39)
-			(end 0.17 -0.39)
+			(start -0.62 -0.39)
+			(end -0.17 -0.39)
 			(stroke
 				(width 0.15)
@@
 		)
 		(fp_line
-			(start 0.62 0.39)
-			(end 0.62 -0.39)
+			(start 0.62 -0.39)
+			(end 0.17 -0.39)
 			(stroke
 				(width 0.15)
@@
 		)
 		(fp_text user "${REFERENCE}"
-			(at 0 -4 0)
+			(at 0 -4 90)
 			(layer "F.SilkS")
 			(effects
@@
 		)
 		(fp_text user "${REFERENCE}"
-			(at 0 -0.25 0)
+			(at 0 -0.25 90)
 			(layer "F.Fab")
 			(effects
@@
 		)
 		(pad "1" smd rect
-			(at -0.24 0)
+			(at -0.24 0 270)
 			(size 0.3 0.32)
 			(layers "F.Cu" "F.Mask" "F.Paste")
@@
 		)
 		(pad "2" smd rect
-			(at 0.24 0)
+			(at 0.24 0 270)
 			(size 0.3 0.32)
 			(layers "F.Cu" "F.Mask" "F.Paste")
@@
 	(footprint "POGO_PAD:POGO_PAD"
 		(layer "F.Cu")
-		(at 0.27 -440)
+		(at -12.5 -8.75)
 		(property "Reference" "REF**"
 			(at 0 -1.5 0)
@@
 	(footprint "POGO_PAD:POGO_PAD"
 		(layer "F.Cu")
-		(at 0.27 -430)
+		(at -11.75 -4.75)
 		(property "Reference" "REF**"
 			(at 0 -1.5 0)
@@
 	(footprint "POGO_PAD:POGO_PAD"
 		(layer "F.Cu")
-		(at 0.27 -420)
+		(at -11.75 -1.75)
 		(property "Reference" "REF**"
 			(at 0 -1.5 0)
@@
 	(footprint "POGO_PAD:POGO_PAD"
 		(layer "F.Cu")
-		(at 0.27 -390)
+		(at -10.75 5)
 		(property "Reference" "REF**"
 			(at 0 -1.5 0)
@@
 	(footprint "POGO_PAD:POGO_PAD"
 		(layer "F.Cu")
-		(at 0.27 -330)
+		(at -10.5 11)
 		(property "Reference" "REF**"
 			(at 0 -1.5 0)
@@
 	(footprint "UNI_ROYAL_0201WMF4701TEE:R0201"
 		(layer "F.Cu")
-		(at 0.27 -510)
+		(at -1.49 -3.75)
 		(property "Reference" "R2"
 			(at 0 -4 0)
