File: layouts/main/main.kicad_pcb (KiCad board)
At the start: 4 copper layers, 20.5 x 20.5 mm, 60 parts, among them U2 MIC_T5838, U5 XCVR_HJ-N54L_SIP

Commit message: wip
Parts:
- renumbered REF** to J_GND, REF** to J_VBAT, U2 to M1, REF** to TP1, REF** to TP10, REF** to TP11, REF** to TP12, REF** to TP13, REF** to TP14, REF** to TP15, REF** to TP2, REF** to TP3, REF** to TP4, REF** to TP5, REF** to TP6, REF** to TP7, REF** to TP8, REF** to TP9
Changed lines of the file:
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@@
 		(layer "F.Cu")
 		(at -6.4 -6.3)
-		(property "Reference" "REF**"
-			(at 0 0 0)
+		(property "Reference" "TP10"
+			(at 0.5 -0.6 0)
 			(layer "F.SilkS")
 			(effects
@@
 		(layer "F.Cu")
 		(at 6.4 5.3)
-		(property "Reference" "REF**"
-			(at 0 0 0)
+		(property "Reference" "TP7"
+			(at 0.6 -0.5 0)
 			(layer "F.SilkS")
 			(effects
@@
 		(layer "F.Cu")
 		(at 5.6 -6.1)
-		(property "Reference" "REF**"
-			(at 0 0 0)
+		(property "Reference" "TP13"
+			(at 0.7 -0.5 0)
 			(layer "F.SilkS")
 			(effects
@@
 		(layer "F.Cu")
 		(at -5.1 -6.3)
-		(property "Reference" "REF**"
-			(at 0 0 0)
+		(property "Reference" "TP11"
+			(at 0.6 -0.7 0)
 			(layer "F.SilkS")
 			(effects
@@
 		(layer "F.Cu")
 		(at 5.2 6.5)
-		(property "Reference" "REF**"
-			(at 0 0 0)
+		(property "Reference" "TP5"
+			(at 0.5 -0.6 0)
 			(layer "F.SilkS")
 			(effects
@@
 		(layer "F.Cu")
 		(at 6.4 6.5)
-		(property "Reference" "REF**"
-			(at 0 0 0)
+		(property "Reference" "TP8"
+			(at 0.6 -0.5 0)
 			(layer "F.SilkS")
 			(effects
@@
 		(layer "F.Cu")
 		(at 4 5.3)
-		(property "Reference" "REF**"
-			(at 0 0 0)
+		(property "Reference" "TP1"
+			(at 0.6 -0.5 0)
 			(layer "F.SilkS")
 			(effects
@@
 		(layer "F.Cu")
 		(at 4 6.5)
-		(property "Reference" "REF**"
-			(at 0.6 -0.2 0)
+		(property "Reference" "TP2"
+			(at 0.6 -0.6 0)
 			(layer "F.SilkS")
 			(effects
@@
 		(layer "F.Cu")
 		(at 4 7.7)
-		(property "Reference" "REF**"
-			(at 0 0 0)
+		(property "Reference" "TP3"
+			(at 0.6 -0.5 0)
 			(layer "F.SilkS")
 			(effects
@@
 		(layer "F.Cu")
 		(at 5.2 5.3)
-		(property "Reference" "REF**"
-			(at -0.5 0 0)
+		(property "Reference" "TP4"
+			(at 0.5 -0.5 0)
 			(layer "F.SilkS")
 			(effects
@@
 		(layer "F.Cu")
 		(at 0.7625 7.662)
-		(property "Reference" "U2"
+		(property "Reference" "M1"
 			(at -0.1625 0 0)
 			(layer "F.SilkS")
@@
 		(layer "F.Cu")
 		(at 6.7 -5.5)
-		(property "Reference" "REF**"
-			(at 0 0 0)
+		(property "Reference" "TP14"
+			(at 0.6 -0.6 0)
 			(layer "F.SilkS")
 			(effects
@@
 		(layer "F.Cu")
 		(at -7.3 -5.3)
-		(property "Reference" "REF**"
-			(at 0 0 0)
+		(property "Reference" "TP9"
+			(at 0 -0.7 0)
 			(layer "F.SilkS")
 			(effects
@@
 		(layer "F.Cu")
 		(at 8.2 -3.6 -90)
-		(property "Reference" "REF**"
-			(at 0 0 90)
+		(property "Reference" "J_GND"
+			(at -0.6 1.4 0)
 			(layer "F.SilkS")
 			(effects
@@
 		(layer "F.Cu")
 		(at -3.8 -6.3)
-		(property "Reference" "REF**"
-			(at 0 0 0)
+		(property "Reference" "TP12"
+			(at 0.4 -0.7 0)
 			(layer "F.SilkS")
 			(effects
@@
 		(layer "F.Cu")
 		(at 5.6 -4.9)
-		(property "Reference" "REF**"
-			(at 0 0 0)
+		(property "Reference" "TP15"
+			(at -0.8 -0.5 0)
 			(layer "F.SilkS")
 			(effects
@@
 		(layer "F.Cu")
 		(at 5.2 7.7)
-		(property "Reference" "REF**"
-			(at 0 0 0)
+		(property "Reference" "TP6"
+			(at 0.5 -0.5 0)
 			(layer "F.SilkS")
 			(effects
@@
 		(layer "F.Cu")
 		(at 8.2 -2 90)
-		(property "Reference" "REF**"
-			(at 0 0 0)
+		(property "Reference" "J_VBAT"
+			(at 0.7 -1.4 0)
 			(layer "F.SilkS")
 			(effects

Commit message: wip
Parts:
- J_GND, J_VBAT: value BATTERY_PAD -> (none)
- M1: value MIC_T5838 -> (none)
- TP1, TP10, TP11, TP12, TP13, TP14, TP15, TP2, TP3, TP4, TP5, TP6, TP7, TP8, TP9: value POGO_PAD -> (none)
- U5: value XCVR_HJ-N54L_SIP -> (none)
Other:
- rule pad_to_mask_clearance: 0.05 -> 0
Changed lines of the file:
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@@
 			(dielectric_constraints no)
 		)
-		(pad_to_mask_clearance 0.05)
+		(pad_to_mask_clearance 0)
 		(solder_mask_min_width 0.1)
 		(allow_soldermask_bridges_in_footprints no)
@@
 			)
 		)
-		(property "Value" "POGO_PAD"
+		(property "Value" ""
 			(at 0 0 0)
 			(layer "F.Fab")
@@
 			)
 		)
-		(property "Value" "POGO_PAD"
+		(property "Value" ""
 			(at 0 0 0)
 			(layer "F.Fab")
@@
 			)
 		)
-		(property "Value" "POGO_PAD"
+		(property "Value" ""
 			(at 0 0 0)
 			(layer "F.Fab")
@@
 			)
 		)
-		(property "Value" "POGO_PAD"
+		(property "Value" ""
 			(at 0 0 0)
 			(layer "F.Fab")
@@
 			)
 		)
-		(property "Value" "POGO_PAD"
+		(property "Value" ""
 			(at 0 0 0)
 			(layer "F.Fab")
@@
 			)
 		)
-		(property "Value" "POGO_PAD"
+		(property "Value" ""
 			(at 0 0 0)
 			(layer "F.Fab")
@@
 			)
 		)
-		(property "Value" "POGO_PAD"
+		(property "Value" ""
 			(at 0 0 0)
 			(layer "F.Fab")
@@
 			)
 		)
-		(property "Value" "POGO_PAD"
+		(property "Value" ""
 			(at 0 0 0)
 			(layer "F.Fab")
@@
 			)
 		)
-		(property "Value" "POGO_PAD"
+		(property "Value" ""
 			(at 0 0 0)
 			(layer "F.Fab")
@@
 			)
 		)
-		(property "Value" "POGO_PAD"
+		(property "Value" ""
 			(at 0 0 0)
 			(layer "F.Fab")
@@
 			)
 		)
-		(property "Value" "MIC_T5838"
+		(property "Value" ""
 			(at -0.1625 0 0)
 			(layer "F.Fab")
@@
 			)
 		)
-		(property "Value" "POGO_PAD"
+		(property "Value" ""
 			(at 0 0 0)
 			(layer "F.Fab")
@@
 			)
 		)
-		(property "Value" "XCVR_HJ-N54L_SIP"
+		(property "Value" ""
 			(at 0 0 0)
 			(layer "F.Fab")
@@
 			)
 		)
-		(property "Value" "POGO_PAD"
+		(property "Value" ""
 			(at 0 0 0)
 			(layer "F.Fab")
@@
 			)
 		)
-		(property "Value" "BATTERY_PAD"
+		(property "Value" ""
 			(at 0 0 90)
 			(layer "F.Fab")
@@
 			)
 		)
-		(property "Value" "POGO_PAD"
+		(property "Value" ""
 			(at 0 0 0)
 			(layer "F.Fab")
@@
 			)
 		)
-		(property "Value" "POGO_PAD"
+		(property "Value" ""
 			(at 0 0 0)
 			(layer "F.Fab")
@@
 			)
 		)
-		(property "Value" "POGO_PAD"
+		(property "Value" ""
 			(at 0 0 0)
 			(layer "F.Fab")
@@
 			)
 		)
-		(property "Value" "BATTERY_PAD"
+		(property "Value" ""
 			(at 0 0 0)
 			(layer "F.Fab")
